Commit message: Imported upstream version '1.1.2' of 'upstream'

File: urdf/zed_descr.urdf.xacro (robot description, xacro)
@@ -24,5 +24,5 @@
   <xacro:arg name="gnss_y" default="0.0" />
   <xacro:arg name="gnss_z" default="0.0" />
-  <xacro:include filename="$(find zed_wrapper)/urdf/zed_macro.urdf.xacro" />
+  <xacro:include filename="$(find zed_description)/urdf/zed_macro.urdf.xacro" />
   <xacro:zed_camera name="$(arg camera_name)" model="$(arg camera_model)" custom_baseline="$(arg custom_baseline)" enable_gnss="$(arg enable_gnss)">
 	    <origin xyz="$(arg gnss_x) $(arg gnss_y) $(arg gnss_z)" rpy="0 0 0"/>

File: urdf/zed_macro.urdf.xacro (robot description, xacro)
@@ -16,5 +16,5 @@
 -->
 <robot xmlns:xacro="http://wiki.ros.org/xacro">
-  <xacro:include filename="$(find zed_wrapper)/urdf/include/materials.urdf.xacro" />
+  <xacro:include filename="$(find zed_description)/urdf/include/materials.urdf.xacro" />
   <xacro:property name="M_PI"     value="3.1415926535897931" />
   <!--
@@ -150,5 +150,5 @@
           <origin xyz="${screw_offset_x} 0 ${screw_offset_z}" rpy="0 0 0"/>
           <geometry>
-            <mesh filename="file://$(find zed_msgs)/meshes/${model}.stl"/>
+            <mesh filename="package://zed_description/meshes/${model}.stl"/>
           </geometry>
           <material name="${model}_mat" />
@@ -157,5 +157,5 @@
           <origin xyz="${screw_offset_x} 0 ${screw_offset_z}" rpy="0 0 0"/>
           <geometry>
-            <mesh filename="file://$(find zed_msgs)/meshes/${model}.stl"/>
+            <mesh filename="package://zed_description/meshes/${model}.stl"/>
           </geometry>
         </collision>
@@ -174,5 +174,5 @@
             <origin xyz="0 0 0" rpy="0 0 0"/>
             <geometry>
-              <mesh filename="file://$(find zed_msgs)/meshes/${model}.stl"/>
+              <mesh filename="package://zed_description/meshes/${model}.stl"/>
             </geometry>
             <material name="${model}_mat" />
@@ -181,5 +181,5 @@
             <origin xyz="0 0 0" rpy="0 0 0"/>
             <geometry>
-              <mesh filename="file://$(find zed_msgs)/meshes/${model}.stl"/>
+              <mesh filename="package://zed_description/meshes/${model}.stl"/>
             </geometry>
           </collision>
@@ -203,5 +203,5 @@
             <origin xyz="0 0 0" rpy="0 0 0"/>
             <geometry>
-              <mesh filename="file://$(find zed_msgs)/meshes/${model}.stl"/>
+              <mesh filename="package://zed_description/meshes/${model}.stl"/>
             </geometry>
             <material name="${model}_mat" />
@@ -210,5 +210,5 @@
             <origin xyz="0 0 0" rpy="0 0 0"/>
             <geometry>
-              <mesh filename="file://$(find zed_msgs)/meshes/${model}.stl"/>
+              <mesh filename="package://zed_description/meshes/${model}.stl"/>
             </geometry>
           </collision>
