Commit message: Imported upstream version '0.1.5' of 'upstream'

File: urdf/zed_macro.urdf.xacro (robot description, xacro)
@@ -16,5 +16,4 @@
 -->
 <robot xmlns:xacro="http://wiki.ros.org/xacro">
-  <xacro:include filename="$(find zed_description)/urdf/include/materials.urdf.xacro" />
   <xacro:property name="M_PI"     value="3.1415926535897931" />
   <!--
@@ -33,4 +32,5 @@
       <xacro:property name="optical_offset_x" value="-0.01" />
       <xacro:property name="mono" value="false" />
+      <xacro:property name="mat" value="0.8 0.8 0.8 1.0" />
     </xacro:if>
     <xacro:if value="${model == 'zedm'}">
@@ -42,4 +42,5 @@
       <xacro:property name="optical_offset_x" value="0.0" />
       <xacro:property name="mono" value="false" />
+      <xacro:property name="mat" value="0 0 0 1.0" />
     </xacro:if>
     <xacro:if value="${model == 'zed2'}">
@@ -51,4 +52,5 @@
       <xacro:property name="optical_offset_x" value="-0.01" />
       <xacro:property name="mono" value="false" />
+      <xacro:property name="mat" value="0.25 0.25 0.25 1.0" />
     </xacro:if>
     <xacro:if value="${model == 'zed2i'}">
@@ -60,4 +62,5 @@
       <xacro:property name="optical_offset_x" value="-0.01" />
       <xacro:property name="mono" value="false" />
+      <xacro:property name="mat" value="0.25 0.25 0.25 1.0" />
     </xacro:if>
     <xacro:if value="${model == 'zedx'}">
@@ -69,4 +72,5 @@
       <xacro:property name="optical_offset_x" value="-0.01" />
       <xacro:property name="mono" value="false" />
+      <xacro:property name="mat" value="0.25 0.25 0.25 1.0" />
     </xacro:if>
     <xacro:if value="${model == 'zedxhdr'}">
@@ -78,4 +82,5 @@
       <xacro:property name="optical_offset_x" value="-0.01" />
       <xacro:property name="mono" value="false" />
+      <xacro:property name="mat" value="0.25 0.25 0.25 1.0" />
     </xacro:if>
     <xacro:if value="${model == 'zedxm'}">
@@ -87,4 +92,15 @@
       <xacro:property name="optical_offset_x" value="-0.01" />
       <xacro:property name="mono" value="false" />
+      <xacro:property name="mat" value="0.25 0.25 0.25 1.0" />
+    </xacro:if>
+    <xacro:if value="${model == 'zedxnano'}">
+      <xacro:property name="baseline" value="0.018" />
+      <xacro:property name="height" value="0.0305" />
+      <xacro:property name="bottom_slope" value="0.0" />
+      <xacro:property name="screw_offset_x" value="0.0" />
+      <xacro:property name="screw_offset_z" value="-0.01525" />
+      <xacro:property name="optical_offset_x" value="-0.01" />
+      <xacro:property name="mono" value="false" />
+      <xacro:property name="mat" value="0.25 0.25 0.25 1.0" />
     </xacro:if>
     <xacro:if value="${model == 'zedxhdrmini'}">
@@ -96,4 +112,5 @@
       <xacro:property name="optical_offset_x" value="-0.01" />
       <xacro:property name="mono" value="false" />
+      <xacro:property name="mat" value="0.25 0.25 0.25 1.0" />
     </xacro:if>
     <xacro:if value="${model == 'zedxhdrmax'}">
@@ -105,4 +122,5 @@
       <xacro:property name="optical_offset_x" value="-0.01" />
       <xacro:property name="mono" value="false" />
+      <xacro:property name="mat" value="0.25 0.25 0.25 1.0" />
     </xacro:if>
     <xacro:if value="${model == 'virtual'}">
@@ -114,4 +132,5 @@
       <xacro:property name="optical_offset_x" value="0.0" />
       <xacro:property name="mono" value="false" />
+      <xacro:property name="mat" value="0.25 0.25 0.25 1.0" />
     </xacro:if>
     <xacro:if value="${model == 'zedxonegs'}">
@@ -121,6 +140,17 @@
       <xacro:property name="screw_offset_x" value="0.0" />
       <xacro:property name="screw_offset_z" value="-0.0155" />
-      <xacro:property name="optical_offset_x" value="0.0" />
+      <xacro:property name="optical_offset_x" value="-0.005" />
       <xacro:property name="mono" value="true" />
+      <xacro:property name="mat" value="0.25 0.25 0.25 1.0" />
+    </xacro:if>
+    <xacro:if value="${model == 'zedxones'}">
+      <xacro:property name="baseline" value="0.0" />
+      <xacro:property name="height" value="0.025" />
+      <xacro:property name="bottom_slope" value="0.0" />
+      <xacro:property name="screw_offset_x" value="0.0" />
+      <xacro:property name="screw_offset_z" value="-0.0125" />
+      <xacro:property name="optical_offset_x" value="0.0" />
+      <xacro:property name="mono" value="true" />
+      <xacro:property name="mat" value="0.25 0.25 0.25 1.0" />
     </xacro:if>
     <xacro:if value="${model == 'zedxone4k'}">
@@ -132,4 +162,5 @@
       <xacro:property name="optical_offset_x" value="0.0" />
       <xacro:property name="mono" value="true" />
+      <xacro:property name="mat" value="0.25 0.25 0.25 1.0" />
     </xacro:if>
     <xacro:if value="${model == 'zedxonehdr'}">
@@ -141,4 +172,5 @@
       <xacro:property name="optical_offset_x" value="0.0" />
       <xacro:property name="mono" value="true" />
+      <xacro:property name="mat" value="0.25 0.25 0.25 1.0" />
     </xacro:if>
     <!-- Camera mounting point (the threaded screw hole in the bottom) -->
@@ -152,5 +184,7 @@
             <mesh filename="package://zed_description/meshes/${model}.stl"/>
           </geometry>
-          <material name="${model}_mat" />
+          <material name="cam_mat">
+            <color rgba="${mat}"/>
+          </material>
         </visual>
         <collision>
@@ -176,5 +210,7 @@
               <mesh filename="package://zed_description/meshes/${model}.stl"/>
             </geometry>
-            <material name="${model}_mat" />
+            <material name="cam_mat">
+              <color rgba="${mat}"/>
+            </material>
           </visual>
           <collision>
@@ -205,5 +241,7 @@
               <mesh filename="package://zed_description/meshes/${model}.stl"/>
             </geometry>
-            <material name="${model}_mat" />
+            <material name="cam_mat">
+              <color rgba="${mat}"/>
+            </material>
           </visual>
           <collision>

Commit message: Rebase from 'upstream'

File: urdf/zed_macro.urdf.xacro (robot description, xacro)
@@ -16,5 +16,4 @@
 -->
 <robot xmlns:xacro="http://wiki.ros.org/xacro">
-  <xacro:include filename="$(find zed_description)/urdf/include/materials.urdf.xacro" />
   <xacro:property name="M_PI"     value="3.1415926535897931" />
   <!--
@@ -33,4 +32,5 @@
       <xacro:property name="optical_offset_x" value="-0.01" />
       <xacro:property name="mono" value="false" />
+      <xacro:property name="mat" value="0.8 0.8 0.8 1.0" />
     </xacro:if>
     <xacro:if value="${model == 'zedm'}">
@@ -42,4 +42,5 @@
       <xacro:property name="optical_offset_x" value="0.0" />
       <xacro:property name="mono" value="false" />
+      <xacro:property name="mat" value="0 0 0 1.0" />
     </xacro:if>
     <xacro:if value="${model == 'zed2'}">
@@ -51,4 +52,5 @@
       <xacro:property name="optical_offset_x" value="-0.01" />
       <xacro:property name="mono" value="false" />
+      <xacro:property name="mat" value="0.25 0.25 0.25 1.0" />
     </xacro:if>
     <xacro:if value="${model == 'zed2i'}">
@@ -60,4 +62,5 @@
       <xacro:property name="optical_offset_x" value="-0.01" />
       <xacro:property name="mono" value="false" />
+      <xacro:property name="mat" value="0.25 0.25 0.25 1.0" />
     </xacro:if>
     <xacro:if value="${model == 'zedx'}">
@@ -69,4 +72,5 @@
       <xacro:property name="optical_offset_x" value="-0.01" />
       <xacro:property name="mono" value="false" />
+      <xacro:property name="mat" value="0.25 0.25 0.25 1.0" />
     </xacro:if>
     <xacro:if value="${model == 'zedxhdr'}">
@@ -78,4 +82,5 @@
       <xacro:property name="optical_offset_x" value="-0.01" />
       <xacro:property name="mono" value="false" />
+      <xacro:property name="mat" value="0.25 0.25 0.25 1.0" />
     </xacro:if>
     <xacro:if value="${model == 'zedxm'}">
@@ -87,4 +92,5 @@
       <xacro:property name="optical_offset_x" value="-0.01" />
       <xacro:property name="mono" value="false" />
+      <xacro:property name="mat" value="0.25 0.25 0.25 1.0" />
     </xacro:if>
     <xacro:if value="${model == 'zedxnano'}">
@@ -96,4 +102,5 @@
       <xacro:property name="optical_offset_x" value="-0.01" />
       <xacro:property name="mono" value="false" />
+      <xacro:property name="mat" value="0.25 0.25 0.25 1.0" />
     </xacro:if>
     <xacro:if value="${model == 'zedxhdrmini'}">
@@ -105,4 +112,5 @@
       <xacro:property name="optical_offset_x" value="-0.01" />
       <xacro:property name="mono" value="false" />
+      <xacro:property name="mat" value="0.25 0.25 0.25 1.0" />
     </xacro:if>
     <xacro:if value="${model == 'zedxhdrmax'}">
@@ -114,4 +122,5 @@
       <xacro:property name="optical_offset_x" value="-0.01" />
       <xacro:property name="mono" value="false" />
+      <xacro:property name="mat" value="0.25 0.25 0.25 1.0" />
     </xacro:if>
     <xacro:if value="${model == 'virtual'}">
@@ -123,4 +132,5 @@
       <xacro:property name="optical_offset_x" value="0.0" />
       <xacro:property name="mono" value="false" />
+      <xacro:property name="mat" value="0.25 0.25 0.25 1.0" />
     </xacro:if>
     <xacro:if value="${model == 'zedxonegs'}">
@@ -132,4 +142,5 @@
       <xacro:property name="optical_offset_x" value="-0.005" />
       <xacro:property name="mono" value="true" />
+      <xacro:property name="mat" value="0.25 0.25 0.25 1.0" />
     </xacro:if>
     <xacro:if value="${model == 'zedxones'}">
@@ -141,4 +152,5 @@
       <xacro:property name="optical_offset_x" value="0.0" />
       <xacro:property name="mono" value="true" />
+      <xacro:property name="mat" value="0.25 0.25 0.25 1.0" />
     </xacro:if>
     <xacro:if value="${model == 'zedxone4k'}">
@@ -150,4 +162,5 @@
       <xacro:property name="optical_offset_x" value="0.0" />
       <xacro:property name="mono" value="true" />
+      <xacro:property name="mat" value="0.25 0.25 0.25 1.0" />
     </xacro:if>
     <xacro:if value="${model == 'zedxonehdr'}">
@@ -159,4 +172,5 @@
       <xacro:property name="optical_offset_x" value="0.0" />
       <xacro:property name="mono" value="true" />
+      <xacro:property name="mat" value="0.25 0.25 0.25 1.0" />
     </xacro:if>
     <!-- Camera mounting point (the threaded screw hole in the bottom) -->
@@ -170,5 +184,7 @@
             <mesh filename="package://zed_description/meshes/${model}.stl"/>
           </geometry>
-          <material name="${model}_mat" />
+          <material name="cam_mat">
+            <color rgba="${mat}"/>
+          </material>
         </visual>
         <collision>
@@ -194,5 +210,7 @@
               <mesh filename="package://zed_description/meshes/${model}.stl"/>
             </geometry>
-            <material name="${model}_mat" />
+            <material name="cam_mat">
+              <color rgba="${mat}"/>
+            </material>
           </visual>
           <collision>
@@ -223,5 +241,7 @@
               <mesh filename="package://zed_description/meshes/${model}.stl"/>
             </geometry>
-            <material name="${model}_mat" />
+            <material name="cam_mat">
+              <color rgba="${mat}"/>
+            </material>
           </visual>
           <collision>
