Commit message: Imported upstream version '0.1.4' of 'upstream'

File: urdf/include/materials.urdf.xacro (robot description, xacro)
@@ -34,4 +34,7 @@
         <color rgba="0.25 0.25 0.25 1.0"/>
     </material>
+    <material name="zedxnano_mat">
+        <color rgba="0.25 0.25 0.25 1.0"/>
+    </material>
     <material name="zedxhdr_mat">
         <color rgba="0.25 0.25 0.25 1.0"/>
@@ -49,4 +52,7 @@
         <color rgba="0.25 0.25 0.25 1.0"/>
     </material>
+    <material name="zedxones_mat">
+        <color rgba="0.25 0.25 0.25 1.0"/>
+    </material>
     <material name="zedxone4k_mat">
         <color rgba="0.25 0.25 0.25 1.0"/>

File: urdf/zed_macro.urdf.xacro (robot description, xacro)
@@ -88,4 +88,13 @@
       <xacro:property name="mono" value="false" />
     </xacro:if>
+    <xacro:if value="${model == 'zedxnano'}">
+      <xacro:property name="baseline" value="0.018" />
+      <xacro:property name="height" value="0.0305" />
+      <xacro:property name="bottom_slope" value="0.0" />
+      <xacro:property name="screw_offset_x" value="0.0" />
+      <xacro:property name="screw_offset_z" value="-0.01525" />
+      <xacro:property name="optical_offset_x" value="-0.01" />
+      <xacro:property name="mono" value="false" />
+    </xacro:if>
     <xacro:if value="${model == 'zedxhdrmini'}">
       <xacro:property name="baseline" value="0.05" />
@@ -121,4 +130,13 @@
       <xacro:property name="screw_offset_x" value="0.0" />
       <xacro:property name="screw_offset_z" value="-0.0155" />
+      <xacro:property name="optical_offset_x" value="-0.005" />
+      <xacro:property name="mono" value="true" />
+    </xacro:if>
+    <xacro:if value="${model == 'zedxones'}">
+      <xacro:property name="baseline" value="0.0" />
+      <xacro:property name="height" value="0.025" />
+      <xacro:property name="bottom_slope" value="0.0" />
+      <xacro:property name="screw_offset_x" value="0.0" />
+      <xacro:property name="screw_offset_z" value="-0.0125" />
       <xacro:property name="optical_offset_x" value="0.0" />
       <xacro:property name="mono" value="true" />

Commit message: Imported upstream version '0.1.3' of 'upstream'

File: urdf/include/materials.urdf.xacro (robot description, xacro)
@@ -34,7 +34,4 @@
         <color rgba="0.25 0.25 0.25 1.0"/>
     </material>
-    <material name="zedxnano_mat">
-        <color rgba="0.25 0.25 0.25 1.0"/>
-    </material>
     <material name="zedxhdr_mat">
         <color rgba="0.25 0.25 0.25 1.0"/>
@@ -52,7 +49,4 @@
         <color rgba="0.25 0.25 0.25 1.0"/>
     </material>
-    <material name="zedxones_mat">
-        <color rgba="0.25 0.25 0.25 1.0"/>
-    </material>
     <material name="zedxone4k_mat">
         <color rgba="0.25 0.25 0.25 1.0"/>

File: urdf/zed_macro.urdf.xacro (robot description, xacro)
@@ -88,13 +88,4 @@
       <xacro:property name="mono" value="false" />
     </xacro:if>
-    <xacro:if value="${model == 'zedxnano'}">
-      <xacro:property name="baseline" value="0.018" />
-      <xacro:property name="height" value="0.0305" />
-      <xacro:property name="bottom_slope" value="0.0" />
-      <xacro:property name="screw_offset_x" value="0.0" />
-      <xacro:property name="screw_offset_z" value="-0.01525" />
-      <xacro:property name="optical_offset_x" value="-0.01" />
-      <xacro:property name="mono" value="false" />
-    </xacro:if>
     <xacro:if value="${model == 'zedxhdrmini'}">
       <xacro:property name="baseline" value="0.05" />
@@ -130,13 +121,4 @@
       <xacro:property name="screw_offset_x" value="0.0" />
       <xacro:property name="screw_offset_z" value="-0.0155" />
-      <xacro:property name="optical_offset_x" value="-0.005" />
-      <xacro:property name="mono" value="true" />
-    </xacro:if>
-    <xacro:if value="${model == 'zedxones'}">
-      <xacro:property name="baseline" value="0.0" />
-      <xacro:property name="height" value="0.025" />
-      <xacro:property name="bottom_slope" value="0.0" />
-      <xacro:property name="screw_offset_x" value="0.0" />
-      <xacro:property name="screw_offset_z" value="-0.0125" />
       <xacro:property name="optical_offset_x" value="0.0" />
       <xacro:property name="mono" value="true" />
